File: pcb/controller/controller.kicad_pcb (KiCad board)
At the start: 2 copper layers, 60 x 70 mm, 39 parts, among them J1 Conn_01x03, J2 Conn_01x03, J3 RELAY_CONN, J4 Remote_header, J5 PWR_IN, J6 MFRC_CONN, J7 Micro_SD_Card, J8 Conn_01x03, J9 Conn_01x03, Q1 MMBT3906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

Commit message: Change footprint to use through-hole, add Edge.cuts cutout for debug pins.
Parts:
- removed J7: Micro_SD_Card, Connector_Card:microSD_HC_Molex_104031-0811
- A1: footprint Module:RaspberryPi_Pico_SMD_HandSolder -> Module:RaspberryPi_Pico_Common_Unspecified
- moved D2 0.05 mm to (88.5, 30.2)
Routing:
- net GND: track 52.6 -> 21.3 mm, vias 14 -> 10
- net GPIO_ACC4: track 91.6 -> 66.4 mm, vias 1 -> 2
- net +3V3: track 208.8 -> 185.2 mm, vias 2 -> 1
- net FLASH_CLK: track 32.7 -> 20.3 mm, vias 1 -> 0
- net FLASH_MOSI: track 28.6 -> 18.4 mm, vias 2 -> 0
- net FLASH_MISO: track 38.9 -> 29.6 mm, vias 1 -> 2
- net FLASH_CS: track 39.4 -> 31.8 mm, vias 3 -> 0
- net FLASH_WP: track 42.4 -> 35.0 mm, vias 1 -> 0
- net GPIO_ACC3: track 45.0 -> 39.0 mm, vias 1 -> 0
- net HEARTBEAT: track 43.0 -> 45.6 mm
- net +5V: track 110.2 -> 112.6 mm, vias 4 -> 3
- net FLASH_HOLD: track 15.6 -> 13.9 mm, vias 1 -> 0
- net GPIO_ACC2: track 54.7 -> 54.9 mm, vias 4 -> 3
Other:
- outline, holes or cut-outs redrawn
- board text added: "Access Control Gen2 LowVolt Controller V1.2"
- board text removed: "Access Control Gen2 LowVolt Controller V1.1"

Commit message: PCB tweaks
Parts:
- moved JP3 1.51 mm to (56.5, 62.9)
Routing:
- net +5V: track 112.6 -> 120.0 mm
- net GPIO_ACC3: track 39.0 -> 42.1 mm
- net +VDC: track 55.6 -> 54.8 mm, vias 1 -> 0
- net +3V3: track 185.2 -> 185.9 mm
Other:
- outline, holes or cut-outs redrawn

Commit message: Update pcby
Routing:
- net +5V: track 120.0 -> 112.1 mm
- net GPIO_ACC3: track 42.1 -> 38.5 mm, vias 0 -> 1
- net GPIO_ACC4: track 66.4 -> 67.1 mm, vias 2 -> 1
Changed lines of the file:
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@@
 	)
 	(segment
-		(start 52.5 72)
-		(end 48.55 68.05)
-		(width 0.6)
-		(layer "B.Cu")
+		(start 50.565686 78.104314)
+		(end 50.565686 68.565686)
+		(width 0.6)
+		(layer "F.Cu")
 		(net "GPIO_ACC3")
 	)
 	(segment
-		(start 48.55 54.55)
-		(end 48.55 68.05)
-		(width 0.6)
-		(layer "B.Cu")
+		(start 45.85 82.82)
+		(end 50.565686 78.104314)
+		(width 0.6)
+		(layer "F.Cu")
 		(net "GPIO_ACC3")
 	)
-	(segment
-		(start 51 81)
-		(end 52.5 79.5)
-		(width 0.6)
-		(layer "B.Cu")
-		(net "GPIO_ACC3")
-	)
-	(segment
-		(start 45.42 51.42)
-		(end 48.55 54.55)
-		(width 0.6)
-		(layer "B.Cu")
-		(net "GPIO_ACC3")
-	)
-	(segment
-		(start 47.67 81)
-		(end 51 81)
-		(width 0.6)
-		(layer "B.Cu")
-		(net "GPIO_ACC3")
-	)
-	(segment
-		(start 52.5 79.5)
-		(end 52.5 72)
-		(width 0.6)
-		(layer "B.Cu")
-		(net "GPIO_ACC3")
-	)
-	(segment
-		(start 45.42 49)
-		(end 45.42 51.42)
-		(width 0.6)
-		(layer "B.Cu")
-		(net "GPIO_ACC3")
-	)
-	(segment
-		(start 45.85 82.82)
-		(end 47.67 81)
-		(width 0.6)
-		(layer "B.Cu")
-		(net "GPIO_ACC3")
-	)
-	(segment
-		(start 47.75 50.01)
-		(end 47.96 49.8)
-		(width 0.4)
-		(layer "F.Cu")
-		(net "GPIO_ACC4")
-	)
-	(segment
-		(start 52 86.622)
-		(end 51.5 86.122)
-		(width 0.6)
-		(layer "F.Cu")
-		(net "GPIO_ACC4")
-	)
-	(segment
-		(start 51.5 86.122)
-		(end 51.5 69.5)
-		(width 0.6)
-		(layer "F.Cu")
-		(net "GPIO_ACC4")
-	)
 	(via
-		(at 52 86.622)
+		(at 50.565686 68.565686)
 		(size 0.6)
 		(drill 0.3)
 		(layers "F.Cu" "B.Cu")
+		(net "GPIO_ACC3")
+	)
+	(segment
+		(start 50.5 68.5)
+		(end 50.565686 68.565686)
+		(width 0.6)
+		(layer "B.Cu")
+		(net "GPIO_ACC3")
+	)
+	(segment
+		(start 45.42 51.42)
+		(end 50.5 56.5)
+		(width 0.6)
+		(layer "B.Cu")
+		(net "GPIO_ACC3")
+	)
+	(segment
+		(start 50.5 56.5)
+		(end 50.5 68.5)
+		(width 0.6)
+		(layer "B.Cu")
+		(net "GPIO_ACC3")
+	)
+	(segment
+		(start 45.42 49)
+		(end 45.42 51.42)
+		(width 0.6)
+		(layer "B.Cu")
+		(net "GPIO_ACC3")
+	)
+	(segment
+		(start 77.28 83)
+		(end 72.83 87.45)
+		(width 0.6)
+		(layer "F.Cu")
+		(net "GPIO_ACC4")
+	)
+	(segment
+		(start 47.75 50.01)
+		(end 47.96 49.8)
+		(width 0.4)
+		(layer "F.Cu")
+		(net "GPIO_ACC4")
+	)
+	(segment
+		(start 52.828 87.45)
+		(end 51.5 86.122)
+		(width 0.6)
+		(layer "F.Cu")
+		(net "GPIO_ACC4")
+	)
+	(segment
+		(start 51.5 86.122)
+		(end 51.5 69.5)
+		(width 0.6)
+		(layer "F.Cu")
+		(net "GPIO_ACC4")
+	)
+	(segment
+		(start 72.83 87.45)
+		(end 52.828 87.45)
+		(width 0.6)
+		(layer "F.Cu")
 		(net "GPIO_ACC4")
 	)
@@
 		(start 51.5 69.5)
 		(end 51.5 55.027208)
-		(width 0.6)
-		(layer "B.Cu")
-		(net "GPIO_ACC4")
-	)
-	(segment
-		(start 77.28 83)
-		(end 73.658 86.622)
-		(width 0.6)
-		(layer "B.Cu")
-		(net "GPIO_ACC4")
-	)
-	(segment
-		(start 73.658 86.622)
-		(end 52 86.622)
 		(width 0.6)
 		(layer "B.Cu")
@@
 	)
 	(segment
-		(start 53 68.5)
-		(end 49.5 68.5)
-		(width 0.6)
-		(layer "F.Cu")
-		(net "+5V")
-	)
-	(segment
-		(start 49.5 68.5)
+		(start 46.25 71.75)
+		(end 53.774859 64.225141)
+		(width 0.6)
+		(layer "F.Cu")
+		(net "+5V")
+	)
+	(segment
+		(start 39.25 71.75)
 		(end 46.25 71.75)
 		(width 0.6)
@@
 	)
 	(segment
+		(start 53.774859 62.225141)
+		(end 54 62)
+		(width 0.6)
+		(layer "F.Cu")
+		(net "+5V")
+	)
+	(segment
+		(start 53.774859 64.225141)
+		(end 53.774859 62.225141)
+		(width 0.6)
+		(layer "F.Cu")
+		(net "+5V")
+	)
+	(segment
 		(start 35.26 35.120456)
 		(end 37.5 37.360456)
@@
 	)
 	(segment
-		(start 46.25 71.75)
-		(end 39.25 71.75)
-		(width 0.6)
-		(layer "F.Cu")
-		(net "+5V")
-	)
-	(segment
 		(start 51.84 51.59)
 		(end 53.75 53.5)
@@
 	)
 	(via
-		(at 53 68.5)
+		(at 54 62)
 		(size 0.6)
 		(drill 0.3)
@@
 	)
 	(segment
-		(start 53.75 67.75)
-		(end 53 68.5)
-		(width 0.6)
-		(layer "B.Cu")
-		(net "+5V")
-	)
-	(segment
 		(start 56.5 53.71)
 		(end 56.29 53.5)
@@
 		(start 56.5 62.2)
 		(end 57.85 62.2)
+		(width 0.6)
+		(layer "B.Cu")
+		(net "+5V")
+	)
+	(segment
+		(start 54 62)
+		(end 56.3 62)
+		(width 0.6)
+		(layer "B.Cu")
+		(net "+5V")
+	)
+	(segment
+		(start 56.3 62)
+		(end 56.5 62.2)
 		(width 0.6)
 		(layer "B.Cu")
@@
 		(layer "B.Cu")
 		(net "+5V")
-	)
-	(segment
-		(start 53.75 53.5)
-		(end 53.75 67.75)
-		(width 0.6)
-		(layer "B.Cu")
-		(net "+5V")

Commit message: Track rerouting
Routing:
- net ACCESS_GRANTED: track 40.1 -> 47.1 mm
- net +3V3: track 185.9 -> 188.9 mm
- net ACCESS_DENIED: track 40.5 -> 41.4 mm

Commit message: More minor PCB tweaks
Parts:
- moved D1 4.00 mm to (63.4, 76.4)
Routing:
- net RELAY+: track 37.9 -> 34.6 mm
- net RELAY-: track 34.6 -> 33.8 mm
- net +5V: track 112.1 -> 111.5 mm
- net +VDC: track 54.8 -> 55.3 mm
Changed lines of the file:
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@@
 	(footprint "Diode_SMD:D_SMA-SMB_Universal_Handsoldering"
 		(layer "F.Cu")
-		(at 59.4 76.42)
+		(at 63.4 76.42)
 		(descr "Diode, Universal, SMA (DO-214AC) or SMB (DO-214AA), Handsoldering,")
 		(tags "Diode Universal SMA (DO-214AC) SMB (DO-214AA) Handsoldering ")
@@
 		)
 	)
-	(gr_text "Access Control Gen2\nLowVolt Controller\nV1.2"
-		(at 59.25 33 0)
+	(gr_text "Access Control Gen2\nLowVolt Controller V1.2"
+		(at 65.25 47 0)
 		(layer "B.SilkS")
 		(effects
@@
 	)
 	(segment
-		(start 63.818522 74.28)
-		(end 61.47 74.28)
-		(width 0.6)
-		(layer "F.Cu")
-		(net "+5V")
-	)
-	(segment
 		(start 35.5 30.66)
 		(end 35.26 30.42)
@@
 	)
 	(segment
-		(start 68.428522 78.89)
-		(end 63.818522 74.28)
-		(width 0.6)
-		(layer "F.Cu")
-		(net "+5V")
-	)
-	(segment
 		(start 38.5 45.5)
 		(end 49.5 45.5)
@@
 	)
 	(via
-		(at 54 62)
+		(at 68.428522 78.89)
 		(size 0.6)
 		(drill 0.3)
@@
 	)
 	(via
-		(at 41.75 76)
+		(at 54 62)
 		(size 0.6)
 		(drill 0.3)
 		(layers "F.Cu" "B.Cu")
-		(capping no)
-		(covering
-			(front no)
-			(back no)
-		)
-		(plugging
-			(front no)
-			(back no)
-		)
-		(filling no)
 		(net "+5V")
 	)
 	(via
-		(at 61.47 74.28)
+		(at 41.75 76)
 		(size 0.6)
 		(drill 0.3)
@@
 	(segment
 		(start 61.47 65.82)
-		(end 61.47 74.28)
+		(end 61.47 72.97)
+		(width 0.6)
+		(layer "B.Cu")
+		(net "+5V")
+	)
+	(segment
+		(start 68.318522 79)
+		(end 68.428522 78.89)
+		(width 0.6)
+		(layer "B.Cu")
+		(net "+5V")
+	)
+	(segment
+		(start 67.5 79)
+		(end 68.318522 79)
 		(width 0.6)
 		(layer "B.Cu")
@@
 	)
 	(segment
+		(start 61.47 72.97)
+		(end 67.5 79)
+		(width 0.6)
+		(layer "B.Cu")
+		(net "+5V")
+	)
+	(segment
 		(start 56.5 62.2)
 		(end 56.5 53.71)
@@
 	)
 	(segment
-		(start 76.75 76.016605)
-		(end 79 78.266605)
-		(width 0.8)
-		(layer "F.Cu")
-		(net "+VDC")
-	)
-	(segment
-		(start 53.75 72.5)
-		(end 53.75 82.22)
-		(width 0.8)
-		(layer "F.Cu")
-		(net "+VDC")
-	)
-	(segment
-		(start 60 70.5)
-		(end 55.5 70.5)
+		(start 55.5 70.5)
+		(end 76 70.5)
 		(width 0.8)
 		(layer "F.Cu")
@@
 	(segment
 		(start 76 70.5)
-		(end 76.75 71.25)
+		(end 78.71 73.21)
 		(width 0.8)
 		(layer "F.Cu")
@@
 	)
 	(segment
-		(start 55.5 70.5)
-		(end 53.75 72.25)
+		(start 53.75 72.5)
+		(end 53.75 82.22)
 		(width 0.8)
 		(layer "F.Cu")
@@
 	)
 	(segment
-		(start 76 70.5)
-		(end 60 70.5)
+		(start 53.75 72.25)
+		(end 55.5 70.5)
 		(width 0.8)
 		(layer "F.Cu")
@@
 	)
 	(segment
-		(start 76.75 71.25)
-		(end 76.75 76.016605)
+		(start 78.71 73.21)
+		(end 78.71 78.89)
 		(width 0.8)
 		(layer "F.Cu")
@@
 	(segment
 		(start 64.83 83.24)
-		(end 63.32 83.24)
-		(width 0.4)
-		(layer "F.Cu")
-		(net "RELAY+")
-	)
-	(segment
-		(start 64.83 83.24)
-		(end 64.07 83.24)
+		(end 64.83 80.75)
 		(width 0.6)
 		(layer "F.Cu")
@@
 	)
 	(segment
-		(start 63.32 83.24)
-		(end 56.5 76.42)
-		(width 0.4)
+		(start 64.83 80.75)
+		(end 60.5 76.42)
+		(width 0.6)
 		(layer "F.Cu")
 		(net "RELAY+")
@@
 	)
 	(segment
-		(start 62.3 76.42)
-		(end 68.33 82.45)
+		(start 66.3 81.21)
+		(end 66.3 76.42)
+		(width 0.6)
+		(layer "F.Cu")
+		(net "RELAY-")
+	)
+	(segment
+		(start 68.33 83.24)
+		(end 66.3 81.21)
 		(width 0.6)
 		(layer "F.Cu")
